File: Tumbler2_Redesign.kicad_pcb (KiCad board)
At the start: 2 copper layers, 0 parts

Commit message: Reset PCB and lock mounting holes
Parts:
- added H1: MountingHole_Pad, MountingHole:MountingHole_3mm_Pad, F.Cu at (119.8, 71.4)
- added H2: MountingHole_Pad, MountingHole:MountingHole_3mm_Pad, F.Cu at (184.8, 71.4)
- added H3: MountingHole_Pad, MountingHole:MountingHole_3mm_Pad, F.Cu at (184.8, 135.4)
- added H4: MountingHole_Pad, MountingHole:MountingHole_3mm_Pad, F.Cu at (119.8, 135.4)
Other:
- board outline added: 77 x 84 mm
