File: Tumbler2_Redesign.kicad_pcb (KiCad board)
At the start: 2 copper layers, 77 x 80.5 mm, 95 parts, among them J1 Conn_01x02, J2 Conn_01x10, J3 Conn_02x08_Odd_Even, J4 USB_C_Receptacle_USB2.0_16P, J5 Conn_01x04, J6 Conn_01x06, J7 Conn_01x06, SW1 SW_Push, SW2 SW_Push, SW3 SW_Push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

Commit message: Prepare for fabrication
Parts:
- moved C13 0.36 mm to (123.7, 140.2)
- moved R14 0.36 mm to (123.7, 142.0)
Routing:
- net 3.3V: track 148.5 -> 143.4 mm, vias 14 -> 12
- net 5V: track 254.7 -> 254.2 mm, vias 5 -> 4
- net GND: vias 216 -> 246

Commit message: Add todo list and update block diagram
Connections:
- J6 pad MP: (no net) -> GND
- J7 pad MP: (no net) -> GND
Changed lines of the file:
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@@
 			(layers "F.Cu" "F.Mask" "F.Paste")
 			(roundrect_rratio 0.138889)
+			(net 1 "GND")
+			(pinfunction "MP")
+			(pintype "passive")
 		)
 		(pad "MP" smd roundrect
@@
 			(layers "F.Cu" "F.Mask" "F.Paste")
 			(roundrect_rratio 0.138889)
+			(net 1 "GND")
+			(pinfunction "MP")
+			(pintype "passive")
 		)
 		(embedded_fonts no)
@@
 			)
 		)
-		(property "Datasheet" "https://www.lcsc.com/datasheet/C191914.pdf"
+		(property "Datasheet" "~"
 			(at 0 0 90)
 			(layer "F.Fab")
@@
 			)
 		)
-		(property "Description" "Connector Header 6 position 2.5mm Pitch 3A Surface Mount, Right Angle -25℃~+85℃"
+		(property "Description" "Generic connector, single row, 01x06, script generated (kicad-library-utils/schlib/autogen/connector/)"
 			(at 0 0 90)
 			(layer "F.Fab")
@@
 			(layers "F.Cu" "F.Mask" "F.Paste")
 			(roundrect_rratio 0.138889)
+			(net 1 "GND")
+			(pinfunction "MP")
+			(pintype "passive")
 		)
 		(pad "MP" smd roundrect
@@
 			(layers "F.Cu" "F.Mask" "F.Paste")
 			(roundrect_rratio 0.138889)
+			(net 1 "GND")
+			(pinfunction "MP")
+			(pintype "passive")
 		)
 		(embedded_fonts no)

Commit message: cleanup schemati, replaced some caps from 0603 to 0805 around Linear Regulator
Parts:
- C1: value 10uF -> 22uF; footprint Capacitor_SMD:C_0603_1608Metric -> Capacitor_SMD:C_0805_2012Metric
- C2, C6, C7: footprint Capacitor_SMD:C_0603_1608Metric -> Capacitor_SMD:C_0805_2012Metric
- R1: value 680 -> 1k
- moved TP2 24.2 mm to (145.3, 78.2)
- moved C7 0.38 mm to (157.9, 96.5)
- moved C1 0.18 mm to (168.0, 94.1)
- moved C6 0.13 mm to (159.9, 96.5)
Routing:
- net GND: track 16.2 -> 18.0 mm
