File: sensors.kicad_sch (KiCad schematic)
At the start: 9 parts, among them J4 Conn_01x04, U10 MPU-6050

Commit message: Remove caps for BTN and GPIO0
Parts:
- renumbered C38 to C36, C39 to C37, C40 to C38
Changed lines of the file:
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@@
 		(dnp no)
 		(fields_autoplaced yes)
-		(property "Reference" "#PWR0130"
+		(property "Reference" "#PWR0128"
 			(at 115.57 119.38 0)
 			(effects
@@
 			(project "Tumbler2_Redesign"
 				(path "/f3fd8d79-9d35-4c04-811e-2697a2740958/38423c09-d546-4c9c-b674-750983dc8f27"
-					(reference "#PWR0130")
+					(reference "#PWR0128")
 					(unit 1)
 				)
@@
 		(dnp no)
 		(fields_autoplaced yes)
-		(property "Reference" "#PWR0122"
+		(property "Reference" "#PWR0120"
 			(at 92.71 81.28 0)
 			(effects
@@
 			(project "Tumbler2_Redesign"
 				(path "/f3fd8d79-9d35-4c04-811e-2697a2740958/38423c09-d546-4c9c-b674-750983dc8f27"
-					(reference "#PWR0122")
+					(reference "#PWR0120")
 					(unit 1)
 				)
@@
 		(dnp no)
 		(fields_autoplaced yes)
-		(property "Reference" "#PWR0127"
+		(property "Reference" "#PWR0125"
 			(at 92.71 97.79 0)
 			(effects
@@
 			(project "Tumbler2_Redesign"
 				(path "/f3fd8d79-9d35-4c04-811e-2697a2740958/38423c09-d546-4c9c-b674-750983dc8f27"
-					(reference "#PWR0127")
+					(reference "#PWR0125")
 					(unit 1)
 				)
@@
 		(dnp no)
 		(fields_autoplaced yes)
-		(property "Reference" "#PWR0131"
+		(property "Reference" "#PWR0129"
 			(at 134.62 119.38 0)
 			(effects
@@
 			(project "Tumbler2_Redesign"
 				(path "/f3fd8d79-9d35-4c04-811e-2697a2740958/38423c09-d546-4c9c-b674-750983dc8f27"
-					(reference "#PWR0131")
+					(reference "#PWR0129")
 					(unit 1)
 				)
@@
 		(dnp no)
 		(fields_autoplaced yes)
-		(property "Reference" "C40"
+		(property "Reference" "C38"
 			(at 172.72 106.6799 0)
 			(effects
@@
 			(project "Tumbler2_Redesign"
 				(path "/f3fd8d79-9d35-4c04-811e-2697a2740958/38423c09-d546-4c9c-b674-750983dc8f27"
-					(reference "C40")
+					(reference "C38")
 					(unit 1)
 				)
@@
 		(dnp no)
 		(fields_autoplaced yes)
-		(property "Reference" "#PWR0124"
+		(property "Reference" "#PWR0122"
 			(at 137.16 81.28 0)
 			(effects
@@
 			(project "Tumbler2_Redesign"
 				(path "/f3fd8d79-9d35-4c04-811e-2697a2740958/38423c09-d546-4c9c-b674-750983dc8f27"
-					(reference "#PWR0124")
+					(reference "#PWR0122")
 					(unit 1)
 				)
@@
 		(dnp no)
 		(fields_autoplaced yes)
-		(property "Reference" "#PWR0133"
+		(property "Reference" "#PWR0131"
 			(at 168.91 119.38 0)
 			(effects
@@
 			(project "Tumbler2_Redesign"
 				(path "/f3fd8d79-9d35-4c04-811e-2697a2740958/38423c09-d546-4c9c-b674-750983dc8f27"
-					(reference "#PWR0133")
+					(reference "#PWR0131")
 					(unit 1)
 				)
@@
 		(dnp no)
 		(fields_autoplaced yes)
-		(property "Reference" "#PWR0125"
+		(property "Reference" "#PWR0123"
 			(at 156.21 81.28 0)
 			(effects
@@
 			(project "Tumbler2_Redesign"
 				(path "/f3fd8d79-9d35-4c04-811e-2697a2740958/38423c09-d546-4c9c-b674-750983dc8f27"
-					(reference "#PWR0125")
+					(reference "#PWR0123")
 					(unit 1)
 				)
@@
 		(dnp no)
 		(fields_autoplaced yes)
-		(property "Reference" "#PWR0129"
+		(property "Reference" "#PWR0127"
 			(at 193.04 107.95 0)
 			(effects
@@
 			(project "Tumbler2_Redesign"
 				(path "/f3fd8d79-9d35-4c04-811e-2697a2740958/38423c09-d546-4c9c-b674-750983dc8f27"
-					(reference "#PWR0129")
+					(reference "#PWR0127")
 					(unit 1)
 				)
@@
 		(dnp no)
 		(fields_autoplaced yes)
-		(property "Reference" "#PWR0132"
+		(property "Reference" "#PWR0130"
 			(at 156.21 119.38 0)
 			(effects
@@
 			(project "Tumbler2_Redesign"
 				(path "/f3fd8d79-9d35-4c04-811e-2697a2740958/38423c09-d546-4c9c-b674-750983dc8f27"
-					(reference "#PWR0132")
+					(reference "#PWR0130")
 					(unit 1)
 				)
@@
 		(dnp no)
 		(fields_autoplaced yes)
-		(property "Reference" "#PWR0123"
+		(property "Reference" "#PWR0121"
 			(at 132.08 81.28 0)
 			(effects
@@
 			(project "Tumbler2_Redesign"
 				(path "/f3fd8d79-9d35-4c04-811e-2697a2740958/38423c09-d546-4c9c-b674-750983dc8f27"
-					(reference "#PWR0123")
+					(reference "#PWR0121")
 					(unit 1)
 				)
@@
 		(dnp no)
 		(fields_autoplaced yes)
-		(property "Reference" "#PWR0128"
+		(property "Reference" "#PWR0126"
 			(at 209.55 102.87 0)
 			(effects
@@
 			(project "Tumbler2_Redesign"
 				(path "/f3fd8d79-9d35-4c04-811e-2697a2740958/38423c09-d546-4c9c-b674-750983dc8f27"
-					(reference "#PWR0128")
+					(reference "#PWR0126")
 					(unit 1)
 				)
@@
 		(dnp no)
 		(fields_autoplaced yes)
-		(property "Reference" "C39"
+		(property "Reference" "C37"
 			(at 160.02 106.6799 0)
 			(effects
@@
 			(project "Tumbler2_Redesign"
 				(path "/f3fd8d79-9d35-4c04-811e-2697a2740958/38423c09-d546-4c9c-b674-750983dc8f27"
-					(reference "C39")
+					(reference "C37")
 					(unit 1)
 				)
@@
 		(dnp no)
 		(fields_autoplaced yes)
-		(property "Reference" "#PWR0126"
+		(property "Reference" "#PWR0124"
 			(at 209.55 90.17 0)
 			(effects
@@
 			(project "Tumbler2_Redesign"
 				(path "/f3fd8d79-9d35-4c04-811e-2697a2740958/38423c09-d546-4c9c-b674-750983dc8f27"
-					(reference "#PWR0126")
+					(reference "#PWR0124")
 					(unit 1)
 				)
@@
 		(on_board yes)
 		(dnp no)
-		(property "Reference" "C38"
+		(property "Reference" "C36"
 			(at 88.9 82.5499 0)
 			(effects
@@
 			(project "Tumbler2_Redesign"
 				(path "/f3fd8d79-9d35-4c04-811e-2697a2740958/38423c09-d546-4c9c-b674-750983dc8f27"
-					(reference "C38")
-					(unit 1)
-				)
+					(reference "C36")
+					(unit 1)
+				)

Commit message: Add missing bus pull-ups
Parts:
- renumbered R17 to R19, R18 to R20, R19 to R21
Changed lines of the file:
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@@
 		(dnp no)
 		(fields_autoplaced yes)
-		(property "Reference" "#PWR0128"
+		(property "Reference" "#PWR0130"
 			(at 115.57 119.38 0)
 			(effects
@@
 			(project "Tumbler2_Redesign"
 				(path "/f3fd8d79-9d35-4c04-811e-2697a2740958/38423c09-d546-4c9c-b674-750983dc8f27"
-					(reference "#PWR0128")
+					(reference "#PWR0130")
 					(unit 1)
 				)
@@
 		(dnp no)
 		(fields_autoplaced yes)
-		(property "Reference" "#PWR0120"
+		(property "Reference" "#PWR0122"
 			(at 92.71 81.28 0)
 			(effects
@@
 			(project "Tumbler2_Redesign"
 				(path "/f3fd8d79-9d35-4c04-811e-2697a2740958/38423c09-d546-4c9c-b674-750983dc8f27"
-					(reference "#PWR0120")
+					(reference "#PWR0122")
 					(unit 1)
 				)
@@
 		(dnp no)
 		(fields_autoplaced yes)
-		(property "Reference" "#PWR0125"
+		(property "Reference" "#PWR0127"
 			(at 92.71 97.79 0)
 			(effects
@@
 			(project "Tumbler2_Redesign"
 				(path "/f3fd8d79-9d35-4c04-811e-2697a2740958/38423c09-d546-4c9c-b674-750983dc8f27"
-					(reference "#PWR0125")
+					(reference "#PWR0127")
 					(unit 1)
 				)
@@
 		(dnp no)
 		(fields_autoplaced yes)
-		(property "Reference" "R19"
+		(property "Reference" "R21"
 			(at 195.58 96.5199 0)
 			(effects
@@
 			(project "Tumbler2_Redesign"
 				(path "/f3fd8d79-9d35-4c04-811e-2697a2740958/38423c09-d546-4c9c-b674-750983dc8f27"
-					(reference "R19")
+					(reference "R21")
 					(unit 1)
 				)
@@
 		(dnp no)
 		(fields_autoplaced yes)
-		(property "Reference" "R17"
+		(property "Reference" "R19"
 			(at 158.75 81.2799 0)
 			(effects
@@
 			(project "Tumbler2_Redesign"
 				(path "/f3fd8d79-9d35-4c04-811e-2697a2740958/38423c09-d546-4c9c-b674-750983dc8f27"
-					(reference "R17")
+					(reference "R19")
 					(unit 1)
 				)
@@
 		(dnp no)
 		(fields_autoplaced yes)
-		(property "Reference" "#PWR0129"
+		(property "Reference" "#PWR0131"
 			(at 134.62 119.38 0)
 			(effects
@@
 			(project "Tumbler2_Redesign"
 				(path "/f3fd8d79-9d35-4c04-811e-2697a2740958/38423c09-d546-4c9c-b674-750983dc8f27"
-					(reference "#PWR0129")
+					(reference "#PWR0131")
 					(unit 1)
 				)
@@
 		(on_board yes)
 		(dnp no)
-		(property "Reference" "R18"
+		(property "Reference" "R20"
 			(at 198.12 86.36 90)
 			(effects
@@
 			(project "Tumbler2_Redesign"
 				(path "/f3fd8d79-9d35-4c04-811e-2697a2740958/38423c09-d546-4c9c-b674-750983dc8f27"
-					(reference "R18")
+					(reference "R20")
 					(unit 1)
 				)
@@
 		(dnp no)
 		(fields_autoplaced yes)
-		(property "Reference" "#PWR0122"
+		(property "Reference" "#PWR0124"
 			(at 137.16 81.28 0)
 			(effects
@@
 			(project "Tumbler2_Redesign"
 				(path "/f3fd8d79-9d35-4c04-811e-2697a2740958/38423c09-d546-4c9c-b674-750983dc8f27"
-					(reference "#PWR0122")
+					(reference "#PWR0124")
 					(unit 1)
 				)
@@
 		(dnp no)
 		(fields_autoplaced yes)
-		(property "Reference" "#PWR0131"
+		(property "Reference" "#PWR0133"
 			(at 168.91 119.38 0)
 			(effects
@@
 			(project "Tumbler2_Redesign"
 				(path "/f3fd8d79-9d35-4c04-811e-2697a2740958/38423c09-d546-4c9c-b674-750983dc8f27"
-					(reference "#PWR0131")
+					(reference "#PWR0133")
 					(unit 1)
 				)
@@
 		(dnp no)
 		(fields_autoplaced yes)
-		(property "Reference" "#PWR0123"
+		(property "Reference" "#PWR0125"
 			(at 156.21 81.28 0)
 			(effects
@@
 			(project "Tumbler2_Redesign"
 				(path "/f3fd8d79-9d35-4c04-811e-2697a2740958/38423c09-d546-4c9c-b674-750983dc8f27"
-					(reference "#PWR0123")
+					(reference "#PWR0125")
 					(unit 1)
 				)
@@
 		(dnp no)
 		(fields_autoplaced yes)
-		(property "Reference" "#PWR0127"
+		(property "Reference" "#PWR0129"
 			(at 193.04 107.95 0)
 			(effects
@@
 			(project "Tumbler2_Redesign"
 				(path "/f3fd8d79-9d35-4c04-811e-2697a2740958/38423c09-d546-4c9c-b674-750983dc8f27"
-					(reference "#PWR0127")
+					(reference "#PWR0129")
 					(unit 1)
 				)
@@
 		(dnp no)
 		(fields_autoplaced yes)
-		(property "Reference" "#PWR0130"
+		(property "Reference" "#PWR0132"
 			(at 156.21 119.38 0)
 			(effects
@@
 			(project "Tumbler2_Redesign"
 				(path "/f3fd8d79-9d35-4c04-811e-2697a2740958/38423c09-d546-4c9c-b674-750983dc8f27"
-					(reference "#PWR0130")
+					(reference "#PWR0132")
 					(unit 1)
 				)
@@
 		(dnp no)
 		(fields_autoplaced yes)
-		(property "Reference" "#PWR0121"
+		(property "Reference" "#PWR0123"
 			(at 132.08 81.28 0)
 			(effects
@@
 			(project "Tumbler2_Redesign"
 				(path "/f3fd8d79-9d35-4c04-811e-2697a2740958/38423c09-d546-4c9c-b674-750983dc8f27"
-					(reference "#PWR0121")
+					(reference "#PWR0123")
 					(unit 1)
 				)
@@
 		(dnp no)
 		(fields_autoplaced yes)
-		(property "Reference" "#PWR0126"
+		(property "Reference" "#PWR0128"
 			(at 209.55 102.87 0)
 			(effects
@@
 			(project "Tumbler2_Redesign"
 				(path "/f3fd8d79-9d35-4c04-811e-2697a2740958/38423c09-d546-4c9c-b674-750983dc8f27"
-					(reference "#PWR0126")
+					(reference "#PWR0128")
 					(unit 1)
 				)
@@
 		(dnp no)
 		(fields_autoplaced yes)
-		(property "Reference" "#PWR0124"
+		(property "Reference" "#PWR0126"
 			(at 209.55 90.17 0)
 			(effects
@@
 			(project "Tumbler2_Redesign"
 				(path "/f3fd8d79-9d35-4c04-811e-2697a2740958/38423c09-d546-4c9c-b674-750983dc8f27"
-					(reference "#PWR0124")
-					(unit 1)
-				)
+					(reference "#PWR0126")
+					(unit 1)
+				)

Commit message: Add expansion pin headers
Parts:
- renumbered J4 to J6
Changed lines of the file:
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@@
 		(on_board yes)
 		(dnp no)
-		(property "Reference" "J4"
+		(property "Reference" "J6"
 			(at 218.44 90.1699 0)
 			(effects
@@
 			(project "Tumbler2_Redesign"
 				(path "/f3fd8d79-9d35-4c04-811e-2697a2740958/38423c09-d546-4c9c-b674-750983dc8f27"
-					(reference "J4")
+					(reference "J6")
 					(unit 1)
 				)
@@
 		(dnp no)
 		(fields_autoplaced yes)
-		(property "Reference" "#PWR0130"
+		(property "Reference" "#PWR0144"
 			(at 115.57 119.38 0)
 			(effects
@@
 			(project "Tumbler2_Redesign"
 				(path "/f3fd8d79-9d35-4c04-811e-2697a2740958/38423c09-d546-4c9c-b674-750983dc8f27"
-					(reference "#PWR0130")
+					(reference "#PWR0144")
 					(unit 1)
 				)
@@
 		(dnp no)
 		(fields_autoplaced yes)
-		(property "Reference" "#PWR0122"
+		(property "Reference" "#PWR0136"
 			(at 92.71 81.28 0)
 			(effects
@@
 			(project "Tumbler2_Redesign"
 				(path "/f3fd8d79-9d35-4c04-811e-2697a2740958/38423c09-d546-4c9c-b674-750983dc8f27"
-					(reference "#PWR0122")
+					(reference "#PWR0136")
 					(unit 1)
 				)
@@
 		(dnp no)
 		(fields_autoplaced yes)
-		(property "Reference" "#PWR0127"
+		(property "Reference" "#PWR0141"
 			(at 92.71 97.79 0)
 			(effects
@@
 			(project "Tumbler2_Redesign"
 				(path "/f3fd8d79-9d35-4c04-811e-2697a2740958/38423c09-d546-4c9c-b674-750983dc8f27"
-					(reference "#PWR0127")
+					(reference "#PWR0141")
 					(unit 1)
 				)
@@
 		(dnp no)
 		(fields_autoplaced yes)
-		(property "Reference" "#PWR0131"
+		(property "Reference" "#PWR0145"
 			(at 134.62 119.38 0)
 			(effects
@@
 			(project "Tumbler2_Redesign"
 				(path "/f3fd8d79-9d35-4c04-811e-2697a2740958/38423c09-d546-4c9c-b674-750983dc8f27"
-					(reference "#PWR0131")
+					(reference "#PWR0145")
 					(unit 1)
 				)
@@
 		(dnp no)
 		(fields_autoplaced yes)
-		(property "Reference" "#PWR0124"
+		(property "Reference" "#PWR0138"
 			(at 137.16 81.28 0)
 			(effects
@@
 			(project "Tumbler2_Redesign"
 				(path "/f3fd8d79-9d35-4c04-811e-2697a2740958/38423c09-d546-4c9c-b674-750983dc8f27"
-					(reference "#PWR0124")
+					(reference "#PWR0138")
 					(unit 1)
 				)
@@
 		(dnp no)
 		(fields_autoplaced yes)
-		(property "Reference" "#PWR0133"
+		(property "Reference" "#PWR0147"
 			(at 168.91 119.38 0)
 			(effects
@@
 			(project "Tumbler2_Redesign"
 				(path "/f3fd8d79-9d35-4c04-811e-2697a2740958/38423c09-d546-4c9c-b674-750983dc8f27"
-					(reference "#PWR0133")
+					(reference "#PWR0147")
 					(unit 1)
 				)
@@
 		(dnp no)
 		(fields_autoplaced yes)
-		(property "Reference" "#PWR0125"
+		(property "Reference" "#PWR0139"
 			(at 156.21 81.28 0)
 			(effects
@@
 			(project "Tumbler2_Redesign"
 				(path "/f3fd8d79-9d35-4c04-811e-2697a2740958/38423c09-d546-4c9c-b674-750983dc8f27"
-					(reference "#PWR0125")
+					(reference "#PWR0139")
 					(unit 1)
 				)
@@
 		(dnp no)
 		(fields_autoplaced yes)
-		(property "Reference" "#PWR0129"
+		(property "Reference" "#PWR0143"
 			(at 193.04 107.95 0)
 			(effects
@@
 			(project "Tumbler2_Redesign"
 				(path "/f3fd8d79-9d35-4c04-811e-2697a2740958/38423c09-d546-4c9c-b674-750983dc8f27"
-					(reference "#PWR0129")
+					(reference "#PWR0143")
 					(unit 1)
 				)
@@
 		(dnp no)
 		(fields_autoplaced yes)
-		(property "Reference" "#PWR0132"
+		(property "Reference" "#PWR0146"
 			(at 156.21 119.38 0)
 			(effects
@@
 			(project "Tumbler2_Redesign"
 				(path "/f3fd8d79-9d35-4c04-811e-2697a2740958/38423c09-d546-4c9c-b674-750983dc8f27"
-					(reference "#PWR0132")
+					(reference "#PWR0146")
 					(unit 1)
 				)
@@
 		(dnp no)
 		(fields_autoplaced yes)
-		(property "Reference" "#PWR0123"
+		(property "Reference" "#PWR0137"
 			(at 132.08 81.28 0)
 			(effects
@@
 			(project "Tumbler2_Redesign"
 				(path "/f3fd8d79-9d35-4c04-811e-2697a2740958/38423c09-d546-4c9c-b674-750983dc8f27"
-					(reference "#PWR0123")
+					(reference "#PWR0137")
 					(unit 1)
 				)
@@
 		(dnp no)
 		(fields_autoplaced yes)
-		(property "Reference" "#PWR0128"
+		(property "Reference" "#PWR0142"
 			(at 209.55 102.87 0)
 			(effects
@@
 			(project "Tumbler2_Redesign"
 				(path "/f3fd8d79-9d35-4c04-811e-2697a2740958/38423c09-d546-4c9c-b674-750983dc8f27"
-					(reference "#PWR0128")
+					(reference "#PWR0142")
 					(unit 1)
 				)
@@
 		(dnp no)
 		(fields_autoplaced yes)
-		(property "Reference" "#PWR0126"
+		(property "Reference" "#PWR0140"
 			(at 209.55 90.17 0)
 			(effects
@@
 			(project "Tumbler2_Redesign"
 				(path "/f3fd8d79-9d35-4c04-811e-2697a2740958/38423c09-d546-4c9c-b674-750983dc8f27"
-					(reference "#PWR0126")
-					(unit 1)
-				)
+					(reference "#PWR0140")
+					(unit 1)
+				)

Commit message: Combine peripheral modules
Parts:
- removed C36, C37: 100nF, Capacitor_SMD:C_0402_1005Metric_Pad0.74x0.62mm_HandSolder, symbol Device:C
- removed C38: 2.2nF, Capacitor_SMD:C_0402_1005Metric_Pad0.74x0.62mm_HandSolder, symbol Device:C
- removed J6: Conn_01x04, Connector_PinHeader_2.54mm:PinHeader_1x04_P2.54mm_Vertical, symbol Connector_Generic:Conn_01x04
- removed R19, R20: 10k, symbol Device:R
- removed R21: 20k, symbol Device:R
- removed TP12: TestPoint, symbol Connector:TestPoint
- removed U10: MPU-6050, Sensor_Motion:InvenSense_QFN-24_4x4mm_P0.5mm, symbol Sensor_Motion:MPU-6050
Connections:
- no-connect marks 2 -> 0
Other:
- note removed: "I2C Address: AD0 tied to GND: 0x68 AD0 tied to VDD: 0x69"
