File: rgb_leds.kicad_sch (KiCad schematic)
At the start: 19 parts

Commit message: Use basic parts where possible
Parts:
- C42, C43, C44, C45, C46, C47, C48, C49, C50, C51: footprint Capacitor_SMD:C_0603_1608Metric_Pad1.08x0.95mm_HandSolder -> Capacitor_SMD:C_0603_1608Metric
- R30: footprint Resistor_SMD:R_0603_1608Metric_Pad0.98x0.95mm_HandSolder -> Resistor_SMD:R_0603_1608Metric; LCSC PN C98220 -> C25804
Changed lines of the file:
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@@
 			)
 		)
-		(property "Footprint" "Capacitor_SMD:C_0603_1608Metric_Pad1.08x0.95mm_HandSolder"
+		(property "Footprint" "Capacitor_SMD:C_0603_1608Metric"
 			(at 139.3952 119.38 0)
 			(effects
@@
 			)
 		)
-		(property "Footprint" "Capacitor_SMD:C_0603_1608Metric_Pad1.08x0.95mm_HandSolder"
+		(property "Footprint" "Capacitor_SMD:C_0603_1608Metric"
 			(at 177.4952 119.38 0)
 			(effects
@@
 			)
 		)
-		(property "Footprint" "Resistor_SMD:R_0603_1608Metric_Pad0.98x0.95mm_HandSolder"
+		(property "Footprint" "Resistor_SMD:R_0603_1608Metric"
 			(at 76.962 73.66 90)
 			(effects
@@
 			)
 		)
-		(property "LCSC PN" "C98220"
+		(property "LCSC PN" "C25804"
 			(at 78.74 73.66 0)
 			(effects
@@
 			)
 		)
-		(property "Footprint" "Capacitor_SMD:C_0603_1608Metric_Pad1.08x0.95mm_HandSolder"
+		(property "Footprint" "Capacitor_SMD:C_0603_1608Metric"
 			(at 113.9952 119.38 0)
 			(effects
@@
 			)
 		)
-		(property "Footprint" "Capacitor_SMD:C_0603_1608Metric_Pad1.08x0.95mm_HandSolder"
+		(property "Footprint" "Capacitor_SMD:C_0603_1608Metric"
 			(at 88.5952 119.38 0)
 			(effects
@@
 			)
 		)
-		(property "Footprint" "Capacitor_SMD:C_0603_1608Metric_Pad1.08x0.95mm_HandSolder"
+		(property "Footprint" "Capacitor_SMD:C_0603_1608Metric"
 			(at 190.1952 119.38 0)
 			(effects
@@
 			)
 		)
-		(property "Footprint" "Capacitor_SMD:C_0603_1608Metric_Pad1.08x0.95mm_HandSolder"
+		(property "Footprint" "Capacitor_SMD:C_0603_1608Metric"
 			(at 126.6952 119.38 0)
 			(effects
@@
 			)
 		)
-		(property "Footprint" "Capacitor_SMD:C_0603_1608Metric_Pad1.08x0.95mm_HandSolder"
+		(property "Footprint" "Capacitor_SMD:C_0603_1608Metric"
 			(at 164.7952 119.38 0)
 			(effects
@@
 			)
 		)
-		(property "Footprint" "Capacitor_SMD:C_0603_1608Metric_Pad1.08x0.95mm_HandSolder"
+		(property "Footprint" "Capacitor_SMD:C_0603_1608Metric"
 			(at 152.0952 119.38 0)
 			(effects
@@
 			)
 		)
-		(property "Footprint" "Capacitor_SMD:C_0603_1608Metric_Pad1.08x0.95mm_HandSolder"
+		(property "Footprint" "Capacitor_SMD:C_0603_1608Metric"
 			(at 202.8952 119.38 0)
 			(effects
@@
 			)
 		)
-		(property "Footprint" "Capacitor_SMD:C_0603_1608Metric_Pad1.08x0.95mm_HandSolder"
+		(property "Footprint" "Capacitor_SMD:C_0603_1608Metric"
 			(at 101.2952 119.38 0)
 			(effects

Commit message: Sketch out component placement
Parts:
- removed C46: 10uF, Capacitor_SMD:C_0603_1608Metric, symbol Device:C
Other:
- moved on the sheet: C42, C43, C44, C45, C47, C48, C49, C50, C51, D10, D3, D4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

Commit message: Continue layout and update schematic
Parts:
- removed C51: 10uF, Capacitor_SMD:C_0603_1608Metric, symbol Device:C
- renumbered C42 to C20, C43 to C21, C44 to C22, C45 to C23, C47 to C24, C48 to C25, C49 to C26, C50 to C27, D7 to D10, D8 to D11, D9 to D12, D10 to D13, D3 to D6, D4 to D7, D5 to D8, D6 to D9, R30 to R24
Other:
- moved on the sheet: C20, C21, C22, C23, C24, C25, C26, C27, D10, D11, D12, D13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

Commit message: Continue layout and add pin header protection
Parts:
- renumbered R24 to R34

Commit message: Document strapping pins
Parts:
- renumbered R34 to R36

Commit message: Connect remaining tracks
Parts:
- renumbered R36 to R28
Changed lines of the file:
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@@
 		(dnp no)
 		(fields_autoplaced yes)
-		(property "Reference" "R36"
+		(property "Reference" "R28"
 			(at 88.9 74.9299 0)
 			(effects
@@
 			(project "Tumbler2_Redesign"
 				(path "/f3fd8d79-9d35-4c04-811e-2697a2740958/8522accb-b87e-46d8-a11d-cbf6de0eac35"
-					(reference "R36")
+					(reference "R28")
 					(unit 1)
 				)
