File: rgb_leds.kicad_sch (KiCad schematic)
At the start: 17 parts

Commit message: cleanup schemati, replaced some caps from 0603 to 0805 around Linear Regulator
Other:
- company: (none) -> ${COMPANY}
- title: (none) -> ${TITLE}
Changed lines of the file:
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@@
 	(generator_version "9.0")
 	(paper "A4")
+	(title_block
+		(title "${TITLE}")
+		(rev "${REVISION}")
+		(company "${COMPANY}")
+		(comment 1 "${AUTHOR1}, ${AUTHOR2}, ${AUTHOR3} ")
+		(comment 2 "Stefan Kummer")
+	)
 	(junction
 		(at 86.36 81.28)
